File: test_hub.sch (KiCad schematic (older format))
At the start: 76 parts

Commit message: First draft of schematic
Parts:
- removed FB? (x5): Ferrite_Bead, symbol Ferrite_Bead
- removed R?: 22, symbol R_Small
- removed U?: MIC550X, symbol MIC550X
- added C14: 1uF, symbol C_Small
- added D1: 3V, symbol LED
- added FB2, FB3, FB4, FB5, FB6: Ferrite_Bead, symbol Ferrite_Bead
- added P2: 5V_SEL, symbol CONN_01X03
- added P3: 5V_EXT, symbol CONN_01X02
- added R12: 22, symbol R_Small
- added R13, R14, R15: 10k, symbol R_Small
- added R16, R19, R22: 100, symbol R_Small
- added R17, R20, R23: R_SNS, symbol R_SNS
- added R18, R21, R24: 0, symbol R_Small
- added R26, R27, R28: 1k, symbol R_Small
- added R29: 680, symbol R_Small
- added R7, R8: 100k, symbol R_Small
- added U2: MIC550X, symbol MIC550X
- added U7, U8, U9: LT6106, symbol LT6106
- D2: renamed from D?; value LED6 -> DBG
- D3: renamed from D?; value LED6 -> 5V_EN3
- D4: renamed from D?; value LED6 -> 5V_EN2
- D5: renamed from D?; value LED6 -> 5V_EN1
- D6: renamed from D?; value LED6 -> LED2
- D7: renamed from D?; value LED6 -> LED1
- D8: renamed from D?; value LED6 -> LED0
- FB1: renamed from FB?; MPN (none) -> BLM18EG221SN1D
- P4: renamed from P?; value USB_A -> USB1
- P5: renamed from P?; value USB_A -> USB2
- P6: renamed from P?; value USB_A -> USB3
- R11: renamed from R?; MPN (none) -> RC0603FR-0722RL
- U1: renamed from U?; MPN (none) -> USB2514B/M2
- U3: renamed from U?; MPN (none) -> STM32F072RBT6
- gave numbers to parts that had none: 55
Connections:
- net LED4 is gone; now on net 5V_EN1: R33.2
- net LED5 is gone; now on net 5V_EN2: R32.2
- net LED6 is gone; now on net 5V_EN3: R31.2
- net LED7 is gone; now on net DBG_LED: R30.2
- net PRT_PWR1 is gone; now on net PRTPWR1: U3.18 (PB0)
- net PRT_PWR2 is gone; now on net PRTPWR2: U3.19 (PB1)
- net PRT_PWR3 is gone; now on net PRTPWR3: U3.20 (PB2)
- net PRT_PWR4 is gone; now on net PRTPWR4: U3.21 (PB10)
- net +3V3: now also R29.2, U2.5 (VOUT)
- net +5V: now also P2.1 (P1), U2.1 (VIN), U2.3 (EN), U7.5 (V+), U8.5 (V+), U9.5 (V+); no longer C16.1, C17.1, C18.1, C19.2, C20.2, C21.2, U4.5 (IN), U5.5 (IN), U6.5 (IN)
- net 5V_EN1: now also U3.34 (PA13), R13.1
- net 5V_EN2: now also U3.37 (PA14), R14.1
- net 5V_EN3: now also U3.38 (PA15), R15.1
- net 5V_FLG1: now also U3.2 (PC13)
- net 5V_FLG2: now also U3.3 (PC14-OSC32_IN)
- net 5V_FLG3: now also U3.4 (PC15-OSC32_OUT)
- net 5V_OUT1: now also FB2.1, R17.3, R18.2; no longer C28.2, C31.1, U4.1 (OUT)
- net 5V_OUT2: now also FB4.1, R20.3, R21.2; no longer C29.2, C32.1, U5.1 (OUT)
- net 5V_OUT3: now also FB6.1, R23.3, R24.2; no longer C30.2, C33.1, U6.1 (OUT)
- net DP4: now also R12.2
- net GND: now also C14.1, D1.1 (K), FB3.1, FB5.1, P3.2 (P2), R13.2, R14.2, R15.2, R26.2, R27.2, R28.2, R8.2, U2.2 (GND), U7.2 (V-), U8.2 (V-), U9.2 (V-)
- net LED0: now also U3.29 (PA8)
- net LED1: now also U3.30 (PA9)
- net LED2: now also U3.31 (PA10)
- net at P6.1 (VCC): now also FB6.2
- net at P6.4 (GND), P6.5 (shield): now also FB5.2
- net VBUS_EXT_DET: now reaches U3.11 (PA1)
- net VBUS_EXT_DET: now also R7.2, R8.1
- net SNS1: now reaches U3.12 (PA2)
- net SNS1: now also R26.1, U7.1 (OUT)
- net SNS2: now reaches U3.13 (PA3)
- net SNS2: now also R27.1, U8.1 (OUT)
- net SNS3: now reaches U3.14 (PA4)
- net SNS3: now also R28.1, U9.1 (OUT)
- net DBG_LED: now reaches U3.28 (PB15)
- net at U3.33 (PA12): now also R12.1
- net at P5.4 (GND), P5.5 (shield): now also FB3.2
- net at P5.1 (VCC): now also FB4.2
- net at P4.1 (VCC): now also FB2.2
- new net: C28.2, C31.1, R17.4, R18.1, U4.1 (OUT)
- new net: C29.2, C32.1, R20.4, R21.1, U5.1 (OUT)
- new net: C30.2, C33.1, R23.4, R24.1, U6.1 (OUT)
- new net: D1.2 (A), R29.1
- new net: R16.1, U7.3 (-IN)
- new net: R16.2, R17.1
- new net: R22.1, U9.3 (-IN)
- new net: R22.2, R23.1
- new net: R19.1, U8.3 (-IN)
- new net: R19.2, R20.1
- new net: R23.2, U9.4 (+IN)
- new net: R20.2, U8.4 (+IN)
- new net: R17.2, U7.4 (+IN)
- new net 5V_EXT: P2.3 (P3), P3.1 (P1)
- new net 5V_OUT: C14.2, C16.1, C17.1, C18.1, C19.2, C20.2, C21.2, P2.2 (P2), R7.1, U4.5 (IN), U5.5 (IN), U6.5 (IN)
- no-connect marks 6 -> 10
Other:
- moved on the sheet: C1, C10, C11, C13, C15, C16, C17, C18, C19, C2, C20, C21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

Commit message: Schematic and footprint assignments done
Parts:
- C1, C10, C11, C12, C13, C14, C15, C19, C2, C20, C21, C22, C23, C24, C25, C26, C27, C28, C29, C3, C30, C4, C5, C6, C7, C8, C9: footprint (none) -> Capacitors_SMD:C_0603
- C16, C17, C18: footprint (none) -> Capacitors_SMD:c_elec_4x5.3
- C31, C32, C33: footprint (none) -> Capacitors_SMD:c_elec_6.3x5.7
- D1, D2, D3, D4, D5, D6, D7, D8: footprint (none) -> LEDs:LED_0603
- FB1, FB2, FB3, FB4, FB5, FB6, R1, R10, R11, R12, R13, R14, R15, R16, R18, R19, R2, R21, R22, R24, R25, R26, R27, R28, R29, R3, R30, R31, R32, R33, R34, R35, R36, R4, R5, R6, R7, R8, R9: footprint (none) -> Resistors_SMD:R_0603
- P1: footprint (none) -> footprints:USB_MICRO_B; MPN 10118192-0001LF -> 10118193-0001LF
- P2: footprint (none) -> Pin_Headers:Pin_Header_Straight_1x03
- P3: footprint (none) -> Pin_Headers:Pin_Header_Straight_1x02
- SW1, SW2: footprint (none) -> footprints:PTS645SM43SMTR92
- U3: footprint (none) -> footprints:LQFP48

Commit message: Fixed schematic bugs and added SWD/UART
Parts:
- added J1: ARM-SWD, footprints:ARM_SWD_SMD, symbol ARM-SWD
- added P7: 5V_SEL, Pin_Headers:Pin_Header_Straight_1x03, symbol CONN_01X03
- P1: footprint footprints:USB_MICRO_B -> footprints:10118193-0001LF
- P4, P5, P6: footprint (none) -> footprints:292303-1
- R17, R20, R23: footprint (none) -> footprints:LVK12
- U1: footprint (none) -> footprints:SQFN36
- U2: footprint (none) -> footprints:SOT-23(M5)
- U4, U5, U6: footprint (none) -> footprints:SOT-25
- U7, U8, U9: footprint (none) -> footprints:TSOT-23-5
- Y1: footprint (none) -> footprints:HCM49
Connections:
- net +3V3: now also U1.21 (OCS_N4), J1.1 (VCC); no longer R25.2
- net 5V_EN1: now also U3.15 (PA5); no longer U3.34 (PA13)
- net 5V_EN2: now also U3.16 (PA6); no longer U3.37 (PA14)
- net 5V_EN3: now also U3.17 (PA7); no longer U3.38 (PA15)
- net GND: now also R25.2, J1.3 (GND), J1.5 (GND), P7.1 (P1)
- net OCS_N1: now also U3.25 (PB12); no longer U3.22 (PB11)
- net OCS_N2: now also U3.26 (PB13); no longer U3.25 (PB12)
- net OCS_N3: now also U3.27 (PB14); no longer U3.26 (PB13)
- net nRST: now also J1.10 (nRESET)
- removed net OCS_N4: U1.21 (OCS_N4), U3.27 (PB14)
- net PRTPWR4: no longer names the net of U1.20 (PRTPWR4/BC_EN4)
- net PRTPWR4: no longer U3.21 (PB10)
- new net SWCLK: J1.4 (SWDCLK/TCK), U3.37 (PA14)
- new net SWDIO: J1.2 (SWDIO/TMS), U3.34 (PA13)
- new net USART3_RX: P7.2 (P2), U3.22 (PB11)
- new net USART3_TX: P7.3 (P3), U3.21 (PB10)
- no-connect marks 10 -> 13

Commit message: PCB routing done (I think)
Parts:
- added C34: 0.1uF, Capacitors_SMD:C_0603, symbol C_Small
- P7: value 5V_SEL -> UART
Connections:
- net +5V: no longer U7.5 (V+), U8.5 (V+), U9.5 (V+)
- net 5V_EN1: now also U3.25 (PB12); no longer U3.15 (PA5)
- net 5V_EN2: now also U3.26 (PB13); no longer U3.16 (PA6)
- net 5V_EN3: now also U3.27 (PB14); no longer U3.17 (PA7)
- net 5V_FLG1: now also U3.29 (PA8); no longer U3.2 (PC13)
- net 5V_FLG2: now also U3.30 (PA9); no longer U3.3 (PC14-OSC32_IN)
- net 5V_FLG3: now also U3.31 (PA10); no longer U3.4 (PC15-OSC32_OUT)
- net 5V_OUT: now also U7.5 (V+), U8.5 (V+), U9.5 (V+)
- net DBG_LED: now also U3.5 (PF0-OSC_IN); no longer U3.28 (PB15)
- net GND: now also C34.1; no longer P1.6 (shield)
- net HUB_RST_N: now also U3.28 (PB15); no longer U3.41 (PB5)
- net LED0: now also U3.2 (PC13); no longer U3.29 (PA8)
- net LED1: now also U3.3 (PC14-OSC32_IN); no longer U3.30 (PA9)
- net LED2: now also U3.4 (PC15-OSC32_OUT); no longer U3.31 (PA10)
- net OCS_N1: now also U3.19 (PB1); no longer U3.25 (PB12)
- net OCS_N2: now also U3.17 (PA7); no longer U3.26 (PB13)
- net OCS_N3: now also U3.15 (PA5); no longer U3.27 (PB14)
- net PRTPWR1: now also U3.20 (PB2); no longer U3.18 (PB0)
- net PRTPWR2: now also U3.18 (PB0); no longer U3.19 (PB1)
- net PRTPWR3: now also U3.16 (PA6); no longer U3.20 (PB2)
- net at FB5.2, P6.4 (GND): no longer P6.5 (shield)
- net at FB3.2, P5.4 (GND): no longer P5.5 (shield)
- net at FB1.2, P4.4 (GND): no longer P4.5 (shield)
- net DM4 renamed USB4_N
- net DM_IN renamed USB_UP_N
- net DN1 renamed USB1_N
- net DN2 renamed USB2_N
- net DN3 renamed USB3_N
- net DP1 renamed USB1_P
- net DP2 renamed USB2_P
- net DP3 renamed USB3_P
- net DP4 renamed USB4_P
- net DP_IN renamed USB_UP_P
- new net GNDPWR: C34.2, P1.6 (shield), P4.5 (shield), P5.5 (shield), P6.5 (shield)

Commit message: Updated MPN's
Parts:
- C22: MPN (none) -> CL21B103KBANNNC
- J1: MPN (none) -> 20021121-00010C4LF
- R2: MPN (none) -> ERJ-3EKF1202V
- SW1, SW2: MPN (none) -> PTS645SM43SMTR92
Changed lines of the file:
@@
 F 2 "Resistors_SMD:R_0603" H 2700 5700 50  0001 C CNN
 F 3 "" H 2700 5700 50  0000 C CNN
+F 4 "ERJ-3EKF1202V" H 2700 5700 60  0001 C CNN "MPN"
 	1    2700 5700
 	1    0    0    -1
@@
 F 2 "footprints:PTS645SM43SMTR92" H 12150 1100 50  0001 C CNN
 F 3 "" H 12150 1100 50  0000 C CNN
+F 4 "PTS645SM43SMTR92" H 12150 1100 60  0001 C CNN "MPN"
 	1    12150 1100
 	1    0    0    -1
@@
 F 2 "footprints:PTS645SM43SMTR92" H 12150 1400 50  0001 C CNN
 F 3 "" H 12150 1400 50  0000 C CNN
+F 4 "PTS645SM43SMTR92" H 12150 1400 60  0001 C CNN "MPN"
 	1    12150 1400
 	1    0    0    -1
@@
 F 2 "Capacitors_SMD:C_0603" H 9450 1300 50  0001 C CNN
 F 3 "" H 9450 1300 50  0000 C CNN
+F 4 "CL21B103KBANNNC" H 9450 1300 60  0001 C CNN "MPN"
 	1    9450 1300
 	-1   0    0    1
@@
 F 2 "footprints:ARM_SWD_SMD" H 14100 1550 60  0001 C CNN
 F 3 "" H 14100 1550 60  0000 C CNN
+F 4 "20021121-00010C4LF" H 14400 1700 60  0001 C CNN "MPN"
 	1    14400 1700
 	1    0    0    -1

Commit message: Kicad version update changes
Parts:
- D1, D2, D3, D4, D5, D6, D7, D8: symbol LED -> LED-RESCUE-test_hub
- FB1, FB2, FB3, FB4, FB5, FB6: symbol Ferrite_Bead -> Ferrite_Bead-RESCUE-test_hub
- P1: symbol USB_OTG -> USB_OTG-RESCUE-test_hub
- P4, P5, P6: symbol USB_A -> USB_A-RESCUE-test_hub
- U7, U8, U9: symbol LT6106 -> LT6106-RESCUE-test_hub
Changed lines of the file:
@@
 EESchema Schematic File Version 2
+LIBS:test_hub-rescue
 LIBS:power
 LIBS:device
@@
 5V_EN3
 $Comp
-L LED D2
+L LED-RESCUE-test_hub D2
 U 1 1 589E4F48
 P 14900 7350
@@
 $EndComp
 $Comp
-L LED D3
+L LED-RESCUE-test_hub D3
 U 1 1 589FCDE2
 P 14900 7650
@@
 $EndComp
 $Comp
-L LED D4
+L LED-RESCUE-test_hub D4
 U 1 1 589FCE96
 P 14900 7950
@@
 $EndComp
 $Comp
-L LED D5
+L LED-RESCUE-test_hub D5
 U 1 1 589FCF49
 P 14900 8250
@@
 $EndComp
 $Comp
-L LED D6
+L LED-RESCUE-test_hub D6
 U 1 1 589FCFFF
 P 14900 8550
@@
 $EndComp
 $Comp
-L LED D7
+L LED-RESCUE-test_hub D7
 U 1 1 589FD0B8
 P 14900 8850
@@
 $EndComp
 $Comp
-L LED D8
+L LED-RESCUE-test_hub D8
 U 1 1 589FD174
 P 14900 9150
@@
 $EndComp
 $Comp
-L USB_A P6
+L USB_A-RESCUE-test_hub P6
 U 1 1 589B30A5
 P 15200 5600
@@
 $EndComp
 $Comp
-L USB_A P5
+L USB_A-RESCUE-test_hub P5
 U 1 1 58A10511
 P 15200 4650
@@
 $EndComp
 $Comp
-L Ferrite_Bead FB1
+L Ferrite_Bead-RESCUE-test_hub FB1
 U 1 1 58A107AC
 P 14500 3350
@@
 $EndComp
 $Comp
-L USB_A P4
+L USB_A-RESCUE-test_hub P4
 U 1 1 58A107B3
 P 15200 3700
@@
 5V_EN3
 $Comp
-L Ferrite_Bead FB2
+L Ferrite_Bead-RESCUE-test_hub FB2
 U 1 1 58A1809C
 P 14500 3900
@@
 $EndComp
 $Comp
-L Ferrite_Bead FB3
+L Ferrite_Bead-RESCUE-test_hub FB3
 U 1 1 58A18194
 P 14500 4300
@@
 $EndComp
 $Comp
-L Ferrite_Bead FB4
+L Ferrite_Bead-RESCUE-test_hub FB4
 U 1 1 58A1828D
 P 14500 4850
@@
 $EndComp
 $Comp
-L Ferrite_Bead FB5
+L Ferrite_Bead-RESCUE-test_hub FB5
 U 1 1 58A1838F
 P 14500 5250
@@
 $EndComp
 $Comp
-L Ferrite_Bead FB6
+L Ferrite_Bead-RESCUE-test_hub FB6
 U 1 1 58A18496
 P 14500 5800
@@
 $EndComp
 $Comp
-L LED D1
+L LED-RESCUE-test_hub D1
 U 1 1 58A2E88C
 P 14900 7050
@@
 $EndComp
 $Comp
-L LT6106 U9
+L LT6106-RESCUE-test_hub U9
 U 1 1 58A50F60
 P 9700 9750
@@
 $EndComp
 $Comp
-L LT6106 U8
+L LT6106-RESCUE-test_hub U8
 U 1 1 58A513CA
 P 9700 8200
@@
 $EndComp
 $Comp
-L LT6106 U7
+L LT6106-RESCUE-test_hub U7
 U 1 1 58A5152E
 P 9700 6550
@@
 Connection ~ 6750 1450
 Wire Wire Line
-	1200 1150 1200 1050
+	1200 1050 1200 1150
 Wire Wire Line
 	9100 4350 8950 4350
@@
 5V_OUT
 $Comp
-L USB_OTG P1
+L USB_OTG-RESCUE-test_hub P1
 U 1 1 589B31ED
 P 1500 7350

Commit message: Adding label for ST usb wires
Connections:
- net ST_USB_N: now reaches R11.1, U3.32 (PA11)
- net ST_USB_P: now reaches R12.1, U3.33 (PA12)
Changed lines of the file:
@@
 	1650 1100 1850 1100
 Connection ~ 1850 1100
+Text Label 9100 4150 2    60   ~ 0
+ST_USB_N
+Text Label 9100 4250 2    60   ~ 0
+ST_USB_P
 $EndSCHEMATC
