File: breakout/hub_breakout.sch (KiCad schematic (older format))
At the start: 48 parts, among them J1 USB_OTG, J2 CONN_01X10, J3 CONN_01X10, J4 CONN_01X02, J5 CONN_01X02, J6 CONN_01X02, J7 CONN_01X02, J8 USB_A, J9 USB_A, U1 MIC550X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

Commit message: Adding BOM for breakout
Parts:
- C10: MPN (none) -> CL10B475KQ8NQNC
- J1: MPN (none) -> 10118193-0001LF
Changed lines of the file:
@@
 LIBS:ostur
 LIBS:test_hub
+LIBS:hub_breakout-cache
 EELAYER 25 0
 EELAYER END
@@
 F 2 "alvarop:USB_MICRO_B" H 1500 5900 50  0001 C CNN
 F 3 "" H 1500 5900 50  0001 C CNN
+F 4 "10118193-0001LF" H 1350 5950 60  0001 C CNN "MPN"
 	1    1350 5950
 	1    0    0    -1
@@
 F 1 "4.7uF" H 4775 1600 50  0000 L CNN
 F 2 "Capacitors_SMD:C_0603" H 4788 1550 50  0001 C CNN
-F 3 "CL10B475KQ8NQNC" H 4750 1700 50  0001 C CNN
+F 3 "" H 4750 1700 50  0001 C CNN
+F 4 "CL10B475KQ8NQNC" H 4750 1700 60  0001 C CNN "MPN"
 	1    4750 1700
 	1    0    0    -1
