File: hw/hub/test_hub.kicad_pcb (KiCad board)
At the start: 2 copper layers, 76.2 x 76.2 mm, 102 parts, among them J1 ARM-SWD, J2 USB_OTG, J3 USB_OTG, J4 USB_A, J5 USB_A, J6 USB_A, P2 5V_SEL, P3 5V_EXT, P7 UART, SW1 RST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

Commit message: Cleaned up silkscreen
Other:
- board text added: "+5"
- board text added: "EXT 5V"
- board text added: "GND"
- board text added: "HOST"
- board text added: "HOST 5V"
Changed lines of the file:
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@@
   (general
     (links 241)
-    (no_connects 3)
+    (no_connects 0)
     (area 76.124999 101.524999 152.475001 177.875001)
     (thickness 1.6)
-    (drawings 45)
+    (drawings 44)
     (tracks 1260)
     (zones 0)
@@
     (tags "capacitor 0603")
     (attr smd)
-    (fp_text reference C5 (at 0 2.794 90) (layer F.SilkS)
+    (fp_text reference C5 (at 2.54 0.127 90) (layer F.SilkS)
       (effects (font (size 1 1) (thickness 0.15)))
     )
@@
   (module footprints:HCM49 (layer F.Cu)
     (at 102.489 156.591)
-    (fp_text reference Y1 (at -7.307 -2.413) (layer F.SilkS)
+    (fp_text reference Y1 (at 0 3.302) (layer F.SilkS)
       (effects (font (size 1 1) (thickness 0.15)))
     )
@@
     (tags "resistor 0603")
     (attr smd)
-    (fp_text reference R2 (at 0 -3.302 270) (layer F.SilkS)
+    (fp_text reference R2 (at -2.413 0 270) (layer F.SilkS)
       (effects (font (size 1 1) (thickness 0.15)))
     )
@@
     (descr "Through hole pin header")
     (tags "pin header")
-    (fp_text reference P2 (at 0 -2.5654) (layer F.SilkS)
+    (fp_text reference P2 (at 0 7.62) (layer F.SilkS)
       (effects (font (size 1 1) (thickness 0.15)))
     )
@@
     (tags "capacitor 0603")
     (attr smd)
-    (fp_text reference C27 (at 0 3.06 90) (layer F.SilkS)
+    (fp_text reference C27 (at 0.127 -2.147 90) (layer F.SilkS)
       (effects (font (size 1 1) (thickness 0.15)))
     )
@@
     (tags "capacitor 0603")
     (attr smd)
-    (fp_text reference C22 (at 0 2.794 90) (layer F.SilkS)
+    (fp_text reference C22 (at 0 1.524 90) (layer F.SilkS)
       (effects (font (size 1 1) (thickness 0.15)))
     )
@@
     (descr "Through hole pin header")
     (tags "pin header")
-    (fp_text reference P7 (at 0 -3.1115 270) (layer F.SilkS)
+    (fp_text reference P7 (at 0 -2.413 270) (layer F.SilkS)
       (effects (font (size 1 1) (thickness 0.15)))
     )
@@
     (tags "capacitor 0603")
     (attr smd)
-    (fp_text reference C30 (at 0 -1.9 270) (layer F.SilkS)
+    (fp_text reference C30 (at -2.286 -0.127 360) (layer F.SilkS)
       (effects (font (size 1 1) (thickness 0.15)))
     )
@@
     (tags "capacitor 0603")
     (attr smd)
-    (fp_text reference C28 (at 0 -1.524 270) (layer F.SilkS)
+    (fp_text reference C28 (at -2.286 -0.127 360) (layer F.SilkS)
       (effects (font (size 1 1) (thickness 0.15)))
     )
@@
     (tags "capacitor 0603")
     (attr smd)
-    (fp_text reference C29 (at -0.012 -1.524 270) (layer F.SilkS)
+    (fp_text reference C29 (at -2.286 -0.127 360) (layer F.SilkS)
       (effects (font (size 1 1) (thickness 0.15)))
     )
@@
     (tags "resistor 0603")
     (attr smd)
-    (fp_text reference FB2 (at 0 -1.9) (layer F.SilkS)
+    (fp_text reference FB2 (at 0 1.651) (layer F.SilkS)
       (effects (font (size 1 1) (thickness 0.15)))
     )
@@
     (tags "capacitor 0603")
     (attr smd)
-    (fp_text reference C26 (at 0.3302 1.4732) (layer F.SilkS)
+    (fp_text reference C26 (at -0.012 1.4732) (layer F.SilkS)
       (effects (font (size 1 1) (thickness 0.15)))
     )
@@
     (tags "resistor 0603")
     (attr smd)
-    (fp_text reference R7 (at 2.968266 -5.223946 270) (layer F.SilkS)
+    (fp_text reference R7 (at 2.286 0 270) (layer F.SilkS)
       (effects (font (size 1 1) (thickness 0.15)))
     )
@@
     (tags "resistor 0603")
     (attr smd)
-    (fp_text reference R8 (at -2.956266 4.461946 450) (layer F.SilkS)
+    (fp_text reference R8 (at -2.286 0 450) (layer F.SilkS)
       (effects (font (size 1 1) (thickness 0.15)))
     )
@@
     (tags "resistor 0603")
     (attr smd)
-    (fp_text reference R9 (at 2.993404 -2.983554 270) (layer F.SilkS)
+    (fp_text reference R9 (at 2.286 0.127 270) (layer F.SilkS)
       (effects (font (size 1 1) (thickness 0.15)))
     )
@@
     (tags "resistor 0603")
     (attr smd)
-    (fp_text reference R10 (at -3.501404 3.745554 270) (layer F.SilkS)
+    (fp_text reference R10 (at -2.794 0 270) (layer F.SilkS)
       (effects (font (size 1 1) (thickness 0.15)))
     )
@@
   (module footprints:LQFP48 (layer F.Cu)
     (at 98.425 119.634 270)
-    (fp_text reference U3 (at -4.826 4.572 360) (layer F.SilkS)
+    (fp_text reference U3 (at -4.318 4.572 360) (layer F.SilkS)
       (effects (font (size 1 1) (thickness 0.15)))
     )
@@
     (tags "resistor 0603")
     (attr smd)
-    (fp_text reference FB8 (at 0 -1.45) (layer F.SilkS)
+    (fp_text reference FB8 (at 0.012 1.524) (layer F.SilkS)
       (effects (font (size 1 1) (thickness 0.15)))
     )
@@
     (tags "resistor 0603")
     (attr smd)
-    (fp_text reference FB10 (at 0 -1.45) (layer F.SilkS)
+    (fp_text reference FB10 (at -0.012 1.524) (layer F.SilkS)
       (effects (font (size 1 1) (thickness 0.15)))
     )
@@
     (tags "resistor 0603")
     (attr smd)
-    (fp_text reference R6 (at -2.274 0 450) (layer F.SilkS)
+    (fp_text reference R6 (at -0.012 -1.524 450) (layer F.SilkS)
       (effects (font (size 1 1) (thickness 0.15)))
     )
@@
     )
   )
+  (gr_text "EXT 5V" (at 106.553 169.164) (layer F.SilkS)
+    (effects (font (size 1.5 1.5) (thickness 0.3)))
+  )
+  (gr_text "HOST 5V" (at 107.442 163.957) (layer F.SilkS)
+    (effects (font (size 1.5 1.5) (thickness 0.3)))
+  )
+  (gr_text GND (at 91.059 160.401) (layer F.SilkS)
+    (effects (font (size 1.5 1.5) (thickness 0.3)))
+  )
+  (gr_text +5 (at 90.424 157.607) (layer F.SilkS)
+    (effects (font (size 1.5 1.5) (thickness 0.3)))
+  )
+  (gr_text PWR (at 82.169 153.797 360) (layer F.SilkS)
+    (effects (font (size 1.5 1.5) (thickness 0.3)))
+  )
+  (gr_text HOST (at 82.677 149.479) (layer F.SilkS)
+    (effects (font (size 1.5 1.5) (thickness 0.3)))
+  )
   (gr_text RST (at 127.635 110.109) (layer B.SilkS)
     (effects (font (size 1.5 1.5) (thickness 0.3)) (justify mirror))
@@
   )
   (gr_line (start 91.059 103.251) (end 91.059 110.109) (layer F.SilkS) (width 0.2))
-  (gr_text USB2 (at 133.858 139.954) (layer F.SilkS)
+  (gr_text USB2 (at 133.985 139.7) (layer F.SilkS)
     (effects (font (size 2 2) (thickness 0.3)))
   )
-  (gr_text USB1 (at 134.112 160.782) (layer F.SilkS)
+  (gr_text USB1 (at 133.985 160.909) (layer F.SilkS)
     (effects (font (size 2 2) (thickness 0.3)))
   )
-  (gr_text ON (at 113.792 152.019) (layer F.SilkS)
+  (gr_text ON (at 114.681 152.908) (layer F.SilkS)
     (effects (font (size 1.5 1.5) (thickness 0.3)))
   )
-  (gr_text ON (at 113.792 130.429) (layer F.SilkS)
+  (gr_text ON (at 114.808 130.683) (layer F.SilkS)
     (effects (font (size 1.5 1.5) (thickness 0.3)))
   )
-  (gr_text ON (at 113.792 108.839) (layer F.SilkS)
+  (gr_text ON (at 114.808 109.093) (layer F.SilkS)
     (effects (font (size 1.5 1.5) (thickness 0.3)))
   )
-  (gr_text "by @alvaroprieto" (at 123.2154 107.1372) (layer F.SilkS)
+  (gr_text "by @alvaroprieto" (at 130.81 106.299) (layer F.SilkS)
     (effects (font (size 1.5 1.5) (thickness 0.3)))
   )
-  (gr_text "USB Test Hub v0.2" (at 122.9106 104.2924) (layer F.SilkS)
+  (gr_text "USB Test Hub v0.2" (at 130.4036 104.0384) (layer F.SilkS)
     (effects (font (size 1.5 1.5) (thickness 0.3)))
   )
-  (gr_text USB3 (at 134.366 118.364) (layer F.SilkS)
+  (gr_text USB3 (at 133.985 118.11) (layer F.SilkS)
     (effects (font (size 2 2) (thickness 0.3)))
   )
@@
     (effects (font (size 4 4) (thickness 1)) (justify mirror))
   )
-  (gr_line (start 80.645 123.571) (end 83.947 124.079) (layer F.SilkS) (width 0.2))
-  (gr_line (start 80.01 124.079) (end 80.01 124.46) (layer F.SilkS) (width 0.2))
-  (gr_line (start 88.138 124.079) (end 80.01 124.079) (layer F.SilkS) (width 0.2))
-  (gr_line (start 88.138 124.46) (end 88.138 124.079) (layer F.SilkS) (width 0.2))
-  (gr_line (start 82.55 123.571) (end 82.55 123.063) (layer F.SilkS) (width 0.2))
-  (gr_line (start 77.089 123.571) (end 82.55 123.571) (layer F.SilkS) (width 0.2))
-  (gr_line (start 77.089 123.063) (end 77.089 123.571) (layer F.SilkS) (width 0.2))
   (gr_text D (at 79.121 119.126) (layer F.SilkS)
     (effects (font (size 1 1) (thickness 0.2)))

Commit message: Testing 4 layer PCB!
Released v0.3 to JLPCB
Parts:
- moved R29 29.8 mm to (59.3, 122.4)
- moved D1 29.8 mm to (56.3, 122.4)
- moved C28 25.4 mm to (103.7, 159.0)
- moved C29 25.4 mm to (103.7, 136.8)
- moved C30 25.4 mm to (103.7, 115.2)
- moved D2 25.4 mm to (56.3, 119.1)
- moved D6 25.4 mm to (56.3, 117.3)
- moved D7 25.4 mm to (56.3, 115.5)
- moved D8 25.4 mm to (56.3, 113.8)
- moved FB5 25.4 mm to (57.7, 158.2)
- moved FB6 25.4 mm to (57.7, 161.0)
- moved J3 25.4 mm to (54.9, 159.6)
- moved P3 25.4 mm to (61.6, 157.7)
- moved R3 25.4 mm to (63.5, 132.6)
- moved R4 25.4 mm to (63.5, 128.0)
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Routing:
- net /5V_OUT: track 271.8 -> 78.3 mm, vias 5 -> 3
- net +3V3: track 185.5 -> 68.3 mm, vias 19 -> 18
- net /5V_EN1: track 158.7 -> 45.0 mm, vias 2 -> 0
- net /5V_FLG1: track 149.8 -> 46.5 mm, vias 2 -> 0
- net /5V_EN2: track 127.2 -> 27.9 mm, vias 2 -> 0
- net /5V_FLG2: track 119.0 -> 29.8 mm, vias 2 -> 0
- net /5V_EN3: track 95.2 -> 35.9 mm, vias 2 -> 0
- net +5V: track 66.7 -> 13.6 mm
- net /5V_FLG3: track 87.9 -> 37.8 mm, vias 2 -> 0
- net /USB3_N: track 70.5 -> 48.6 mm, vias 0 -> 1
- net /USB3_P: track 70.4 -> 48.6 mm, vias 0 -> 1
- net /USB2_P: track 59.0 -> 42.2 mm, vias 0 -> 1
- net /USB2_N: track 59.0 -> 42.2 mm, vias 0 -> 1
- net GND: track 115.0 -> 126.3 mm, vias 46 -> 48
- net /USB_UP_N: track 28.1 -> 20.4 mm, vias 0 -> 2
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- added copper zone on Power, net +3V3
- added copper zone on Power, net +5V
- added copper zone on Power, net /5V_OUT
- added copper zone on Ground, net GND
- removed copper zone on B.Cu, net GND
Other:
- copper layers 2 -> 4
- rule pad_to_mask_clearance: 0.2 -> 0.0508
- board text added: "USB Test Hub v0.3"
- board text removed: "USB Test Hub v0.2"
